File: project_b2_vouhnouta24/.history/project_b2_vouhnouta24.kicad_sch (KiCad schematic)
At the start: 5 parts, among them U1 ATmega328-P, Y1 16Mhz

Commit message: some progress
gonna finish at home
Parts:
- added J1: AVR-ISP-10, symbol Connector:AVR-ISP-10
- added R1: 10M, symbol Device:R
Connections:
- net +5V: now also J1.2 (VCC), R1.2
- net Earth: now also U1.22 (GND), U1.8 (GND), J1.10 (GND), J1.4 (GND), J1.6 (GND), J1.8 (GND); no longer Y1.1, Y1.2
- net at C2.2, U1.10 (XTAL2/PB7): now also Y1.2
- net at U1.1 (~{RESET}/PC6): now also J1.5 (~{RST}), R1.1
- net at C3.2, U1.9 (XTAL1/PB6): now also Y1.1
Other:
- moved on the sheet: Y1

Commit message: custom U1
Parts:
- U1: value ATmega328-P -> ATmega328-P-A
Connections:
- net +5V: now also U1.18 (AVCC); no longer U1.20 (AVCC)
- net Earth: now also U1.3 (GND); no longer U1.8 (GND)
- net at C2.2, Y1.2: now also U1.8 (XTAL2/PB7); no longer U1.10 (XTAL2/PB7)
- net at C3.2, Y1.1: now also U1.7 (XTAL1/PB6); no longer U1.9 (XTAL1/PB6)
- net at C1.1: now also U1.20 (AREF); no longer U1.21 (AREF)
- new net: R1.1, U1.29 (~{RESET}/PC6)
- now unconnected: J1.5 (~{RST}), U1.1 (~{RESET}/PC6)
Changed lines of the file:
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@@
 	(paper "A3" portrait)
-	(junction
-		(at 161.29 196.85)
-		(diameter 0)
-		(color 0 0 0 0)
-	)
 	(junction
 		(at 170.18 173.99)
@@
 	(wire
 		(pts
+			(xy 245.11 182.88) (xy 247.65 182.88)
+		)
+		(stroke
+			(width 0)
+			(type default)
+		)
+	)
+	(wire
+		(pts
 			(xy 196.85 196.85) (xy 173.99 196.85)
 		)
@@
 	(wire
 		(pts
-			(xy 161.29 199.39) (xy 228.6 199.39)
+			(xy 245.11 187.96) (xy 247.65 187.96)
 		)
 		(stroke
@@
 	(wire
 		(pts
-			(xy 245.11 190.5) (xy 246.38 190.5)
-		)
-		(stroke
-			(width 0)
-			(type default)
-		)
-	)
-	(wire
-		(pts
-			(xy 246.38 199.39) (xy 236.22 199.39)
-		)
-		(stroke
-			(width 0)
-			(type default)
-		)
-	)
-	(wire
-		(pts
-			(xy 161.29 196.85) (xy 161.29 199.39)
+			(xy 245.11 190.5) (xy 247.65 190.5)
 		)
 		(stroke
@@
 	(wire
 		(pts
-			(xy 161.29 196.85) (xy 166.37 196.85)
+			(xy 160.02 196.85) (xy 166.37 196.85)
 		)
 		(stroke
@@
 	(wire
 		(pts
-			(xy 228.6 203.2) (xy 228.6 199.39)
-		)
-		(stroke
-			(width 0)
-			(type default)
-		)
-	)
-	(wire
-		(pts
-			(xy 236.22 203.2) (xy 228.6 203.2)
-		)
-		(stroke
-			(width 0)
-			(type default)
-		)
-	)
-	(wire
-		(pts
 			(xy 170.18 186.69) (xy 196.85 186.69)
 		)
@@
 	(wire
 		(pts
-			(xy 246.38 199.39) (xy 246.38 190.5)
-		)
-		(stroke
-			(width 0)
-			(type default)
-		)
-	)
-	(wire
-		(pts
 			(xy 170.18 170.18) (xy 170.18 173.99)
 		)
@@
 		)
 	)
-	(wire
-		(pts
-			(xy 236.22 199.39) (xy 236.22 203.2)
-		)
-		(stroke
-			(width 0)
-			(type default)
-		)
-	)
 	(bus
 		(pts
@@
 	(wire
 		(pts
+			(xy 245.11 185.42) (xy 247.65 185.42)
+		)
+		(stroke
+			(width 0)
+			(type default)
+		)
+	)
+	(wire
+		(pts
 			(xy 170.18 176.53) (xy 171.45 176.53)
-		)
-		(stroke
-			(width 0)
-			(type default)
-		)
-	)
-	(wire
-		(pts
-			(xy 160.02 196.85) (xy 161.29 196.85)
 		)
 		(stroke
@@
 			)
 		)
-		(property "Value" "ATmega328-P"
+		(property "Value" "ATmega328-P-A"
 			(at 162.306 150.114 0)
 			(show_name no)
@@
 		)
 		(property "Footprint" "Package_DIP:DIP-28_W7.62mm"
-			(at 144.78 189.23 0)
+			(at 77.216 201.422 0)
 			(hide yes)
 			(show_name no)
@@
 		)
 		(property "Datasheet" "http://ww1.microchip.com/downloads/en/DeviceDoc/ATmega328_P%20AVR%20MCU%20with%20picoPower%20Technology%20Data%20Sheet%2040001984A.pdf"
-			(at 144.78 189.23 0)
+			(at 61.722 239.268 0)
 			(hide yes)
 			(show_name no)
@@
 		)
 		(property "Description" "20MHz, 32kB Flash, 2kB SRAM, 1kB EEPROM, DIP-28"
-			(at 144.78 189.23 0)
+			(at 83.312 211.328 0)
 			(hide yes)
 			(show_name no)
@@
 		(pin "4"
 		)
-		(pin "5"
+		(pin "32"
 		)
 		(pin "23"
@@
 		(pin "12"
 		)
-		(pin "6"
+		(pin "30"
 		)
 		(pin "1"
@@
 		(pin "20"
 		)
-		(pin "21"
+		(pin "29"
 		)
 		(pin "16"
@@
 		(pin "9"
 		)
-		(pin "19"
+		(pin "31"
 		)
 		(pin "25"

Commit message: implemented U1
Connections:
- net at C2.2, Y1.2: no longer U1.8 (XTAL2/PB7)
- net at R1.1: now also U1.19 (ADC6); no longer U1.29 (~{RESET}/PC6)
- net at C3.2, Y1.1: now also U1.8 (XTAL2/PB7); no longer U1.7 (XTAL1/PB6)
Changed lines of the file:
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@@
 		(pin "26"
+		)
+		(pin "6"
+		)
+		(pin "5"
+		)
+		(pin "21"
+		)
+		(pin "19"
+		)
+		(pin "22"
 		)
 		(instances
