File: project_b2_vouhnouta24/.history/project_b2_vouhnouta24.kicad_sch (KiCad schematic)
At the start: 7 parts, among them J1 AVR-ISP-10, U1 ATmega328-P-A, Y1 16Mhz

Commit message: completely fixed J1
A lot of broke moving it around and trying to figure out the bus connections.
Connections:
- net RST: now reaches J1.5 (~{RST})
- net RST: now also R1.1, U1.19 (ADC6), U1.29 (~{RESET}/PC6)
Other:
- moved on the sheet: J1
Changed lines of the file:
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@@
+	)
+	(junction
+		(at 163.83 196.85)
+		(diameter 0)
+		(color 0 0 0 0)
+	)
+	(junction
+		(at 163.83 193.04)
+		(diameter 0)
+		(color 0 0 0 0)
 	)
 	(junction
@@
 	)
 	(bus_entry
-		(at 256.54 190.5)
+		(at 256.54 185.42)
+		(size 2.54 2.54)
+		(stroke
+			(width 0)
+			(type default)
+		)
+	)
+	(bus_entry
+		(at 175.26 194.31)
 		(size 2.54 -2.54)
 		(stroke
@@
 		)
 	)
-	(bus_entry
-		(at 256.54 185.42)
-		(size 2.54 -2.54)
-		(stroke
-			(width 0)
-			(type default)
-		)
-	)
-	(bus_entry
-		(at 256.54 187.96)
-		(size 2.54 -2.54)
-		(stroke
-			(width 0)
-			(type default)
-		)
-	)
-	(bus_entry
-		(at 256.54 182.88)
-		(size 2.54 -2.54)
-		(stroke
-			(width 0)
-			(type default)
-		)
-	)
 	(wire
 		(pts
@@
 	(wire
 		(pts
-			(xy 245.11 182.88) (xy 256.54 182.88)
+			(xy 245.11 193.04) (xy 256.54 193.04)
 		)
 		(stroke
@@
 	(wire
 		(pts
+			(xy 171.45 179.07) (xy 175.26 179.07)
+		)
+		(stroke
+			(width 0)
+			(type default)
+		)
+	)
+	(wire
+		(pts
+			(xy 196.85 186.69) (xy 196.85 175.26)
+		)
+		(stroke
+			(width 0)
+			(type default)
+		)
+	)
+	(wire
+		(pts
+			(xy 160.02 196.85) (xy 163.83 196.85)
+		)
+		(stroke
+			(width 0)
+			(type default)
+		)
+	)
+	(wire
+		(pts
+			(xy 245.11 185.42) (xy 256.54 185.42)
+		)
+		(stroke
+			(width 0)
+			(type default)
+		)
+	)
+	(wire
+		(pts
+			(xy 163.83 193.04) (xy 163.83 196.85)
+		)
+		(stroke
+			(width 0)
+			(type default)
+		)
+	)
+	(wire
+		(pts
+			(xy 160.02 173.99) (xy 170.18 173.99)
+		)
+		(stroke
+			(width 0)
+			(type default)
+		)
+	)
+	(wire
+		(pts
+			(xy 245.11 190.5) (xy 256.54 190.5)
+		)
+		(stroke
+			(width 0)
+			(type default)
+		)
+	)
+	(bus
+		(pts
+			(xy 259.08 165.1) (xy 259.08 199.39)
+		)
+		(stroke
+			(width 0)
+			(type default)
+		)
+	)
+	(wire
+		(pts
+			(xy 196.85 162.56) (xy 196.85 175.26)
+		)
+		(stroke
+			(width 0)
+			(type default)
+		)
+	)
+	(wire
+		(pts
+			(xy 160.02 193.04) (xy 163.83 193.04)
+		)
+		(stroke
+			(width 0)
+			(type default)
+		)
+	)
+	(wire
+		(pts
+			(xy 171.45 176.53) (xy 171.45 179.07)
+		)
+		(stroke
+			(width 0)
+			(type default)
+		)
+	)
+	(wire
+		(pts
+			(xy 167.64 194.31) (xy 175.26 194.31)
+		)
+		(stroke
+			(width 0)
+			(type default)
+		)
+	)
+	(wire
+		(pts
 			(xy 245.11 187.96) (xy 256.54 187.96)
 		)
@@
 	(wire
 		(pts
-			(xy 245.11 190.5) (xy 256.54 190.5)
-		)
-		(stroke
-			(width 0)
-			(type default)
-		)
-	)
-	(wire
-		(pts
-			(xy 171.45 179.07) (xy 175.26 179.07)
-		)
-		(stroke
-			(width 0)
-			(type default)
-		)
-	)
-	(wire
-		(pts
-			(xy 196.85 186.69) (xy 196.85 175.26)
-		)
-		(stroke
-			(width 0)
-			(type default)
-		)
-	)
-	(wire
-		(pts
-			(xy 160.02 196.85) (xy 166.37 196.85)
-		)
-		(stroke
-			(width 0)
-			(type default)
-		)
-	)
-	(wire
-		(pts
-			(xy 160.02 173.99) (xy 170.18 173.99)
-		)
-		(stroke
-			(width 0)
-			(type default)
-		)
-	)
-	(wire
-		(pts
-			(xy 196.85 162.56) (xy 196.85 175.26)
-		)
-		(stroke
-			(width 0)
-			(type default)
-		)
-	)
-	(wire
-		(pts
-			(xy 171.45 176.53) (xy 171.45 179.07)
+			(xy 163.83 196.85) (xy 166.37 196.85)
+		)
+		(stroke
+			(width 0)
+			(type default)
+		)
+	)
+	(wire
+		(pts
+			(xy 167.64 193.04) (xy 167.64 194.31)
 		)
 		(stroke
@@
 	(wire
 		(pts
-			(xy 245.11 185.42) (xy 256.54 185.42)
-		)
-		(stroke
-			(width 0)
-			(type default)
-		)
-	)
-	(wire
-		(pts
 			(xy 170.18 176.53) (xy 171.45 176.53)
 		)
@@
 		)
 	)
-	(bus
-		(pts
-			(xy 259.08 177.8) (xy 259.08 199.39)
+	(wire
+		(pts
+			(xy 163.83 193.04) (xy 167.64 193.04)
 		)
 		(stroke
@@
 		)
 	)
-	(label "MISO"
-		(at 250.19 182.88 0)
+	(label "RST"
+		(at 252.73 185.42 0)
 		(effects
 			(font
@@
 		)
 	)
-	(label "SCK"
-		(at 250.19 187.96 0)
+	(label "RST"
+		(at 172.72 194.31 0)
 		(effects
 			(font
@@
 		)
 	)
+	(label "MISO"
+		(at 252.73 193.04 0)
+		(effects
+			(font
+				(size 1.27 1.27)
+			)
+			(justify left bottom)
+		)
+	)
 	(label "MOSI"
-		(at 250.19 185.42 0)
+		(at 252.73 190.5 0)
+		(effects
+			(font
+				(size 1.27 1.27)
+			)
+			(justify left bottom)
+		)
+	)
+	(label "SCK"
+		(at 252.73 187.96 0)
 		(effects
 			(font
@@
 		(lib_id "Connector:AVR-ISP-10")
 		(at 234.95 187.96 0)
+		(mirror x)
 		(unit 1)
 		(body_style 1)
@@
 		(in_pos_files yes)
 		(dnp no)
-		(fields_autoplaced yes)
 		(property "Reference" "J1"
-			(at 226.06 185.4199 0)
+			(at 226.06 190.5001 0)
 			(show_name no)
 			(do_not_autoplace no)
@@
 		)
 		(property "Value" "AVR-ISP-10"
-			(at 226.06 187.9599 0)
+			(at 226.06 187.9601 0)
 			(show_name no)
 			(do_not_autoplace no)
@@
 		)
 		(property "Footprint" ""
-			(at 228.6 186.69 90)
+			(at 228.6 189.23 90)
 			(hide yes)
 			(show_name no)
@@
 		)
 		(property "Datasheet" ""
-			(at 202.565 201.93 0)
+			(at 202.565 173.99 0)
 			(hide yes)
 			(show_name no)
@@
 	(symbol
 		(lib_id "power:+5V")
-		(at 232.41 175.26 0)
+		(at 232.41 200.66 180)
 		(unit 1)
 		(body_style 1)
@@
 		(fields_autoplaced yes)
 		(property "Reference" "#PWR05"
-			(at 232.41 179.07 0)
+			(at 232.41 196.85 0)
 			(hide yes)
 			(show_name no)
@@
 		)
 		(property "Value" "+5V"
-			(at 232.41 170.18 0)
-			(show_name no)
-			(do_not_autoplace no)
-			(effects
-				(font
-					(size 1.27 1.27)
-				)
+			(at 234.95 201.9299 0)
+			(show_name no)
+			(do_not_autoplace no)
+			(effects
+				(font
+					(size 1.27 1.27)
+				)
+				(justify right)
 			)
 		)
 		(property "Footprint" ""
-			(at 232.41 175.26 0)
+			(at 232.41 200.66 0)
 			(hide yes)
 			(show_name no)
@@
 		)
 		(property "Datasheet" ""
-			(at 232.41 175.26 0)
+			(at 232.41 200.66 0)
 			(hide yes)
 			(show_name no)
@@
 		)
 		(property "Description" "Power symbol creates a global label with name \"+5V\""
-			(at 232.41 175.26 0)
+			(at 232.41 200.66 0)
 			(hide yes)
 			(show_name no)
@@
 	(symbol
 		(lib_id "power:Earth")
-		(at 232.41 198.12 0)
+		(at 232.41 177.8 180)
 		(unit 1)
 		(body_style 1)
@@
 		(dnp no)
 		(property "Reference" "#PWR06"
-			(at 232.41 204.47 0)
+			(at 232.41 171.45 0)
 			(hide yes)
 			(show_name no)
@@
 		)
 		(property "Value" "Earth"
-			(at 232.41 202.184 0)
+			(at 232.41 173.736 0)
 			(show_name no)
 			(do_not_autoplace no)
@@
 		)
 		(property "Footprint" ""
-			(at 232.41 198.12 0)
+			(at 232.41 177.8 0)
 			(hide yes)
 			(show_name no)
@@
 		)
 		(property "Datasheet" ""
-			(at 232.41 198.12 0)
+			(at 232.41 177.8 0)
 			(hide yes)
 			(show_name no)
@@
 		)
 		(property "Description" "Power symbol creates a global label with name \"Earth\""
-			(at 232.41 198.12 0)
-			(hide yes)
-			(show_name no)
+			(at 232.41 177.8 0)
+			(hide yes)
+			(show_name no)

Commit message: J1 bus complete
Parts:
- added U2: ADP2108AUJ-3.3, Package_TO_SOT_SMD:TSOT-23-5, symbol Regulator_Switching:ADP2108AUJ-3.3
Connections:
- net MISO: now also U1.16 (PB4)
- net MOSI: now also U1.15 (PB3)
- net SCK: now also U1.17 (PB5)
Other:
- moved on the sheet: C2, C3, J1, Y1

Commit message: U2 modulator
Parts:
- added C4: 4.7u, Capacitor_THT:CP_Radial_D6.3mm_P2.50mm, symbol Device:C_Polarized
- added C5: 10u, Capacitor_THT:CP_Radial_D6.3mm_P2.50mm, symbol Device:C_Polarized
- added L1: 1u, Inductor_SMD:L_2010_5025Metric, symbol Device:L
Connections:
- net +5V: now also U2.1 (Vin), U2.3 (EN), C4.1
- net Earth: now also U2.2 (GND), C4.2, C5.2
- net +3.3V: now reaches U2.4 (FB)
- net +3.3V: now also C5.1, L1.2
- net at U2.5 (SW): now also L1.1
Other:
- moved on the sheet: U2

Commit message: SD card start
Parts:
- added J2: Micro_SD_Card, symbol Connector:Micro_SD_Card
- added U3: TXB0104D, Package_SO:SOIC-14_3.9x8.7mm_P1.27mm, symbol Logic_LevelTranslator:TXB0104D
Connections:
- net +5V: now also U3.1 (VCCA), U3.8 (OE)
- net Earth: now also J2.6 (VSS), U3.7 (GND)
- new net: J2.3 (CMD), U3.12 (B2)
- new net: J2.2 (DAT3/CD), U3.13 (B1)
- new net +3.3VA: J2.4 (VDD), U3.14 (VCCB)
Other:
- moved on the sheet: C4, C5, L1, U2

Commit message: all the busses connected correctly finally
Connections:
- net +3.3VA is gone; now on net +3.3V: J2.4 (VDD), U3.14 (VCCB)
- net MISO: now also U3.5 (A4)
- net MOSI: now also U3.3 (A2)
- net SCK: now also U3.4 (A3)
- net at C2.2, Y1.2: now also U1.23 (PC0)
- net at U3.10 (B4): now also J2.7 (DAT0)
- net at U3.11 (B3): now also J2.5 (CLK)
- net CS: now reaches U3.2 (A1)
- net CS: now also U1.14 (PB2)
Other:
- moved on the sheet: C1, J2, U1, U3

Commit message: displaybus
Parts:
- added DS1: HY1602E, Display:HY1602E, symbol Display_Character:HY1602E
- added R2: 120R, Resistor_SMD:R_0805_2012Metric, symbol Device:R
- added R3, R4: 10k, Resistor_SMD:R_0805_2012Metric, symbol Device:R
- added SW1: RotaryEncoder, symbol Device:RotaryEncoder
Connections:
- net +5V: now also DS1.4 (VDD), R2.2, R3.2, R4.1
- net Earth: now also DS1.1 (LEDK), DS1.3 (VSS), DS1.5 (Vo), SW1.C
- net at C2.2, Y1.2: now also U1.7 (XTAL1/PB6); no longer U1.23 (PC0)
- net DB3: now reaches U1.1 (PD3)
- net DB3: now also DS1.12 (DB3)
- net DB6: now reaches U1.10 (PD6)
- net DB6: now also DS1.15 (DB6)
- net DB7: now reaches U1.11 (PD7)
- net DB7: now also DS1.16 (DB7)
- net ENC_A: now reaches U1.12 (PB0)
- net ENC_A: now also R3.1, SW1.A
- net ENC_B: now reaches U1.13 (PB1)
- net ENC_B: now also R4.2, SW1.B
- net DB4: now reaches U1.2 (PD4)
- net DB4: now also DS1.13 (DB4)
- net LCD_RW: now reaches U1.24 (PC1)
- net LCD_RW: now also DS1.7 (R/~{W})
- net LCD_RS: now reaches U1.25 (PC2)
- net LCD_RS: now also DS1.6 (RS)
- net DB0: now reaches U1.30 (PD0)
- net DB0: now also DS1.9 (DB0)
- net DB1: now reaches U1.31 (PD1)
- net DB1: now also DS1.10 (DB1)
- net DB2: now reaches U1.32 (PD2)
- net DB2: now also DS1.11 (DB2)
- net DB5: now reaches U1.9 (PD5)
- net DB5: now also DS1.14 (DB5)
- new net: DS1.2 (LEDA), R2.1
- new net LCD_E: DS1.8 (E), U1.23 (PC0)

Commit message: Final product
It is probably dysfunctional but i did not have any more time in class. gg
Parts:
- added C6, C7: 100n, Capacitor_SMD:C_0805_2012Metric, symbol Device:C
Connections:
- net +5V: now also U1.4 (VCC), U1.6 (VCC), C6.2, C7.2
- net Earth: now also C6.1, C7.1
